File: tiny_solar_supply.kicad_pcb (KiCad board)
At the start: 2 copper layers, 33.9 x 14.2 mm, 17 parts, among them J1 Conn_01x02_Pin, J2 Conn_01x02_Pin, J3 Conn_01x02_Pin, J4 Conn_01x02_Pin, Q1 2N7002, U1 AP3015AKTR-G1

Commit message: Optimization
Parts:
- L1: footprint ASPI-0630LR-100M-T15:IND_ASPI-0630LR_ABR -> ASPI-0630LR-100M-T15:IND_ASPI-0630LR_ABR-M
- moved C2 11.2 mm to (198.3, 110.2)
- moved C3 9.28 mm to (196.9, 100.4), turned to 0 degrees
- moved R1 7.29 mm to (191.9, 100.3), turned to 0 degrees
- moved L1 3.43 mm to (190.8, 107.1), turned to 180 degrees
- moved J1 2.43 mm to (199.9, 106.5), turned to 180 degrees
- moved U1 0.91 mm to (183.1, 104.9), turned to -90 degrees
- moved R3 0.54 mm to (179.7, 105.2)
- moved C1 0.50 mm to (181.0, 109.7)
- moved R2 0.39 mm to (183.1, 109.7), turned to -90 degrees
- moved R4 0.30 mm to (176.9, 105.2), turned to 90 degrees
- moved J2 0.22 mm to (170.3, 100.6)
- moved J4 0.22 mm to (170.3, 106.8)
- moved J3 0.10 mm to (173.9, 100.6)
Routing:
- net GNDD: track 64.9 -> 1.09 mm, vias 0 -> 19
- net Net-(D1-A): track 34.0 -> 19.3 mm
- net Net-(J3-Pin_2): track 37.0 -> 22.5 mm, vias 2 -> 3
- net Net-(U1-FB): track 13.9 -> 28.2 mm
- net /OUT_P: track 31.8 -> 21.6 mm
- net Net-(Q1-D): track 11.4 -> 5.79 mm
- net /SOLAR_P: track 11.3 -> 10.3 mm
- added copper zone on F.Cu, net GNDD
