File: tiny_solar_supply.kicad_sch (KiCad schematic)
At the start: 16 parts, among them J1 Conn_01x02_Pin, J2 Conn_01x02_Pin, J3 Conn_01x02_Pin, J4 Conn_01x02_Pin, Q1 2N7002, U1 AP3015AKTR-G1

Commit message: Optimization
Parts:
- L1: footprint ASPI-0630LR-100M-T15:IND_ASPI-0630LR_ABR -> ASPI-0630LR-100M-T15:IND_ASPI-0630LR_ABR-M
Changed lines of the file:
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@@
 			)
 		)
-		(property "Footprint" "ASPI-0630LR-100M-T15:IND_ASPI-0630LR_ABR"
+		(property "Footprint" "ASPI-0630LR-100M-T15:IND_ASPI-0630LR_ABR-M"
 			(at 109.22 71.12 0)
 			(hide yes)
@@
 			(show_name no)
 			(do_not_autoplace no)
+			(effects
+				(font
+					(size 1.27 1.27)
+				)
+			)
+		)
+		(property "Purpose" ""
+			(at 109.22 71.12 0)
+			(show_name no)
+			(do_not_autoplace no)
